File: hardware/elec/eagle-9.5.1/HUM-ASM-001/HUM-ASM-001-v0-1.sch (EAGLE design)
At the start: 11 parts

Commit message: * finished building pcb library parts * added one of each part to schematic * added Power and Audio pages to schematic
Parts:
- added C1: (no value), MG-Eagle_v1:CAP_THT_POL-E-035X080MM
- added J1: B2B-XH-AM(LF)(SN), MG-Eagle_v1:CON_JST_2-PIN_B2B-XH-AM
- added J2: 75869-131LF, MG-Eagle_v1:CON_HEADER_2X3SHROUD
- added LED1: (no value), MG-Eagle_v1:LED_THT-3MM
- added U1: MCP23017-E/SP, MG-Eagle_v1:IIC_MCP23017-E/SP
- K1, K2: value (none) -> 7-1393239-7
- Q1, Q2: value (none) -> IRLB8721PBF
- THM-1: value (none) -> 532702B02500G
- THM-2: value (none) -> V5629W220
- VRG-1: value (none) -> NID100-5
Other:
- note added: "Audio"
- note added: "MCU"
- note added: "Power"
Changed lines of the file:
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@@
 <part name="ASM-3" library="MG-Eagle_v1" deviceset="ASM_ADAFRUIT_MAX98306_AMP" device=""/>
 <part name="ASM-4" library="MG-Eagle_v1" deviceset="ASM_ADAFRUIT_INA169" device=""/>
-<part name="VRG-1" library="MG-Eagle_v1" deviceset="VRG_NID100" device=""/>
-<part name="K1" library="MG-Eagle_v1" deviceset="EMD_RELAY_SPDT_8-PIN" device="_TE_7-1393239-7"/>
-<part name="K2" library="MG-Eagle_v1" deviceset="EMD_RELAY_SPDT_8-PIN" device="_TE_7-1393239-7"/>
-<part name="Q1" library="MG-Eagle_v1" deviceset="TRN_MOSFET-N" device="_TO-220_VERTICAL"/>
-<part name="Q2" library="MG-Eagle_v1" deviceset="TRN_MOSFET-N" device="_TO-220_VERTICAL"/>
-<part name="THM-1" library="MG-Eagle_v1" deviceset="THM_HEATSINK_2-PIN" device=""/>
-<part name="THM-2" library="MG-Eagle_v1" deviceset="THM_HEATSINK_1-PIN" device="" package3d_urn="urn:adsk.eagle:package:14183/1"/>
+<part name="K1" library="MG-Eagle_v1" deviceset="EMD_RELAY_SPDT_8-PIN" device="_TE_7-1393239-7" value="7-1393239-7"/>
+<part name="K2" library="MG-Eagle_v1" deviceset="EMD_RELAY_SPDT_8-PIN" device="_TE_7-1393239-7" value="7-1393239-7"/>
+<part name="Q1" library="MG-Eagle_v1" deviceset="TRN_MOSFET-N" device="_TO-220_VERTICAL" value="IRLB8721PBF"/>
+<part name="Q2" library="MG-Eagle_v1" deviceset="TRN_MOSFET-N" device="_TO-220_VERTICAL" value="IRLB8721PBF"/>
+<part name="THM-1" library="MG-Eagle_v1" deviceset="THM_HEATSINK_2-PIN" device="" value="532702B02500G"/>
+<part name="THM-2" library="MG-Eagle_v1" deviceset="THM_HEATSINK_1-PIN" device="" package3d_urn="urn:adsk.eagle:package:14183/1" value="V5629W220"/>
+<part name="J1" library="MG-Eagle_v1" deviceset="CON_JST_2-PIN" device="_B2B-XH-AM" value="B2B-XH-AM(LF)(SN)"/>
+<part name="LED1" library="MG-Eagle_v1" deviceset="LED_THT" device="-3MM"/>
+<part name="J2" library="MG-Eagle_v1" deviceset="CON_HEADER_2X3" device="SHROUD" value="75869-131LF"/>
+<part name="U1" library="MG-Eagle_v1" deviceset="IIC_MCP23017-E/SP" device="" value="MCP23017-E/SP"/>
+<part name="C1" library="MG-Eagle_v1" deviceset="CAP_THT_POL" device="-E-035X080MM"/>
+<part name="FRAME4" library="MG-Eagle_v1" deviceset="SCH_FRAME_LETTER_8.5X11" device="">
+<attribute name="CNAME" value="HumidiFire"/>
+<attribute name="CREVISION" value="1.0"/>
+<attribute name="DESIGNER" value="Matt Garfield"/>
+</part>
+<part name="VRG-1" library="MG-Eagle_v1" deviceset="VRG_NID100" device="" value="NID100-5"/>
+<part name="FRAME2" library="MG-Eagle_v1" deviceset="SCH_FRAME_LETTER_8.5X11" device="">
+<attribute name="CNAME" value="HumidiFire"/>
+<attribute name="CREVISION" value="1.0"/>
+<attribute name="DESIGNER" value="Matt Garfield"/>
+</part>
 </parts>
 <sheets>
 <sheet>
+<description>MCU</description>
 <plain>
+<text x="162.56" y="-172.72" size="5.08" layer="97" font="vector">MCU</text>
 </plain>
 <instances>
-<instance part="FRAME1" gate="G$1" x="0" y="0" smashed="yes">
-<attribute name="DRAWING_NAME" x="167.64" y="-182.88" size="1.778" layer="94" font="vector"/>
-<attribute name="LAST_DATE_TIME" x="167.64" y="-187.96" size="2.286" layer="94" font="vector"/>
-<attribute name="SHEET" x="181.61" y="-193.04" size="2.54" layer="94" font="vector"/>
-<attribute name="CNAME" x="167.64" y="-177.8" size="2.54" layer="94" font="vector"/>
-<attribute name="CREVISION" x="226.03" y="-193.14" size="2.54" layer="94" font="vector"/>
-<attribute name="DESIGNER" x="217.37" y="-187.96" size="2.54" layer="94" font="vector"/>
+<instance part="FRAME1" gate="G$1" x="-2.54" y="0" smashed="yes">
+<attribute name="DRAWING_NAME" x="165.1" y="-182.88" size="1.778" layer="94" font="vector"/>
+<attribute name="LAST_DATE_TIME" x="165.1" y="-187.96" size="2.286" layer="94" font="vector"/>
+<attribute name="SHEET" x="179.07" y="-193.04" size="2.54" layer="94" font="vector"/>
+<attribute name="CNAME" x="165.1" y="-177.8" size="2.54" layer="94" font="vector"/>
+<attribute name="CREVISION" x="223.49" y="-193.14" size="2.54" layer="94" font="vector"/>
+<attribute name="DESIGNER" x="214.83" y="-187.96" size="2.54" layer="94" font="vector"/>
 </instance>
 <instance part="ASM-1" gate="G$1" x="33.02" y="-40.64" smashed="yes">
 <attribute name="NAME" x="17.78" y="-10.16" size="1.778" layer="95" align="top-left"/>
-<attribute name="VALUE" x="17.78" y="-63.5" size="1.778" layer="96" align="top-left"/>
+<attribute name="VALUE" x="17.78" y="-63.5" size="1.27" layer="96" align="top-left"/>
 </instance>
 <instance part="ASM-2" gate="G$1" x="86.36" y="-43.18" smashed="yes">
@@
 <attribute name="NAME" x="182.88" y="-21.59" size="1.778" layer="95" font="vector"/>
 </instance>
-<instance part="VRG-1" gate="G$1" x="231.14" y="-124.46" smashed="yes">
-<attribute name="VALUE" x="223.52" y="-146.304" size="1.27" layer="96" font="vector" align="top-left"/>
-<attribute name="NAME" x="223.52" y="-105.41" size="1.778" layer="95" font="vector"/>
-</instance>
 <instance part="K1" gate="G$1" x="33.02" y="-116.84" smashed="yes">
 <attribute name="NAME" x="22.86" y="-103.632" size="1.778" layer="95"/>
-<attribute name="VALUE" x="22.86" y="-132.08" size="1.778" layer="96"/>
+<attribute name="VALUE" x="22.86" y="-132.08" size="1.27" layer="96"/>
 </instance>
 <instance part="K2" gate="G$1" x="33.02" y="-149.86" smashed="yes">
 <attribute name="NAME" x="22.86" y="-136.652" size="1.778" layer="95"/>
-<attribute name="VALUE" x="22.86" y="-165.1" size="1.778" layer="96"/>
+<attribute name="VALUE" x="22.86" y="-165.1" size="1.27" layer="96"/>
 </instance>
 <instance part="Q1" gate="G$1" x="106.68" y="-116.84" smashed="yes">
 <attribute name="NAME" x="111.76" y="-114.3" size="1.778" layer="95" font="vector"/>
-<attribute name="VALUE" x="111.76" y="-116.84" size="1.27" layer="96" font="vector" ratio="12"/>
+<attribute name="VALUE" x="111.76" y="-116.84" size="1.27" layer="96" font="vector"/>
 </instance>
 <instance part="Q2" gate="G$1" x="106.68" y="-132.08" smashed="yes">
 <attribute name="NAME" x="111.76" y="-129.54" size="1.778" layer="95" font="vector"/>
-<attribute name="VALUE" x="111.76" y="-132.08" size="1.27" layer="96" font="vector" ratio="12"/>
+<attribute name="VALUE" x="111.76" y="-132.08" size="1.27" layer="96" font="vector"/>
 </instance>
 <instance part="THM-1" gate="G$1" x="152.4" y="-127" smashed="yes">
 <attribute name="NAME" x="158.115" y="-123.825" size="1.778" layer="95"/>
-<attribute name="VALUE" x="158.115" y="-126.365" size="1.778" layer="96"/>
+<attribute name="VALUE" x="158.115" y="-126.365" size="1.27" layer="96"/>
 </instance>
 <instance part="THM-2" gate="G$1" x="152.4" y="-142.24" smashed="yes">
 <attribute name="NAME" x="158.115" y="-139.065" size="1.778" layer="95"/>
-<attribute name="VALUE" x="158.115" y="-141.605" size="1.778" layer="96"/>
+<attribute name="VALUE" x="158.115" y="-141.605" size="1.27" layer="96"/>
+</instance>
+<instance part="J1" gate="G$1" x="152.4" y="-106.68" smashed="yes">
+<attribute name="NAME" x="149.86" y="-100.838" size="1.778" layer="95"/>
+<attribute name="VALUE" x="149.86" y="-111.76" size="1.27" layer="96" font="vector"/>
+</instance>
+<instance part="LED1" gate="G$1" x="175.26" y="-93.98" smashed="yes">
+<attribute name="NAME" x="171.196" y="-97.409" size="1.778" layer="95" font="vector"/>
+<attribute name="VALUE" x="171.196" y="-98.298" size="1.27" layer="96" font="vector" ratio="12" align="top-left"/>
+</instance>
+<instance part="J2" gate="G$1" x="114.3" y="-160.02" smashed="yes">
+<attribute name="NAME" x="109.22" y="-154.432" size="1.778" layer="95"/>
+<attribute name="VALUE" x="109.22" y="-167.132" size="1.27" layer="96"/>
+</instance>
+<instance part="U1" gate="G$1" x="223.52" y="-50.8" smashed="yes">
+<attribute name="NAME" x="213.3406" y="-21.7935" size="1.7814" layer="95"/>
+<attribute name="VALUE" x="214.371509375" y="-81.5479" size="1.27" layer="96"/>
+</instance>
+<instance part="C1" gate="G$1" x="119.38" y="-83.82" smashed="yes">
+<attribute name="NAME" x="120.396" y="-83.185" size="1.778" layer="95" ratio="10"/>
+<attribute name="VALUE" x="120.396" y="-88.011" size="1.27" layer="96" font="vector"/>
 </instance>
 </instances>
+<busses>
+</busses>
+<nets>
+</nets>
+</sheet>
+<sheet>
+<description>Power</description>
+<plain>
+<text x="165.1" y="-172.72" size="5.08" layer="97" font="vector">Power</text>
+</plain>
+<instances>
+<instance part="FRAME4" gate="G$1" x="0" y="0" smashed="yes">
+<attribute name="DRAWING_NAME" x="167.64" y="-182.88" size="1.778" layer="94" font="vector"/>
+<attribute name="LAST_DATE_TIME" x="167.64" y="-187.96" size="2.286" layer="94" font="vector"/>
+<attribute name="SHEET" x="181.61" y="-193.04" size="2.54" layer="94" font="vector"/>
+<attribute name="CNAME" x="167.64" y="-177.8" size="2.54" layer="94" font="vector"/>
+<attribute name="CREVISION" x="226.03" y="-193.14" size="2.54" layer="94" font="vector"/>
+<attribute name="DESIGNER" x="217.37" y="-187.96" size="2.54" layer="94" font="vector"/>
+</instance>
+<instance part="VRG-1" gate="G$1" x="101.6" y="-81.28" smashed="yes">
+<attribute name="VALUE" x="93.98" y="-103.124" size="1.27" layer="96" font="vector" align="top-left"/>
+<attribute name="NAME" x="93.98" y="-62.23" size="1.778" layer="95" font="vector"/>
+</instance>
+</instances>
+<busses>
+</busses>
+<nets>
+</nets>
+</sheet>
+<sheet>
+<description>Audio</description>
+<plain>
+<text x="165.1" y="-172.72" size="5.08" layer="97" font="vector">Audio</text>
+</plain>
+<instances>
+<instance part="FRAME2" gate="G$1" x="0" y="0" smashed="yes">
+<attribute name="DRAWING_NAME" x="167.64" y="-182.88" size="1.778" layer="94" font="vector"/>
+<attribute name="LAST_DATE_TIME" x="167.64" y="-187.96" size="2.286" layer="94" font="vector"/>
+<attribute name="SHEET" x="181.61" y="-193.04" size="2.54" layer="94" font="vector"/>
+<attribute name="CNAME" x="167.64" y="-177.8" size="2.54" layer="94" font="vector"/>
+<attribute name="CREVISION" x="226.03" y="-193.14" size="2.54" layer="94" font="vector"/>
+<attribute name="DESIGNER" x="217.37" y="-187.96" size="2.54" layer="94" font="vector"/>
+</instance>
+</instances>

Commit message: * Major progress on schematic
Parts:
- added D1: 1N4001, MG-Eagle_v1:DIO_DIODEPTH
- added J10, J11, J12: (no value), MG-Eagle_v1:CON_HEADER_1X4NO_SILK_ALL_ROUND
- added J13, J14: (no value), MG-Eagle_v1:CON_HEADER_1X31X03_NO_SILK
- added J15, J16, J20: (no value), MG-Eagle_v1:CON_HEADER_1X21X02_NO_SILK
- added J17, J18: (no value), MG-Eagle_v1:CON_HEADER_1X1-QC_TAB_121786-1
- added J19: (no value), MG-Eagle_v1:CON_HEADER_1X5NO_SILK
- added J3: (no value), MG-Eagle_v1:CON_HEADER_1X16-1X16_NO_SILK
- added J4: (no value), MG-Eagle_v1:CON_HEADER_1X12_NO_SILK
- added J5, J6, J7, J8: (no value), MG-Eagle_v1:CON_HEADER_1X14
- added J9: (no value), MG-Eagle_v1:CON_HEADER_1X7NO_SILK
- added JP1, JP2, JP3, JP4, JP5, JP6, JP7, JP8: CON_JUMPER_PAD-2-NC_BY_TRACE, MG-Eagle_v1:CON_JUMPER_PAD-2-NC_BY_TRACE
- added R1: 1k, MG-Eagle_v1:RES_RESISTOR-PTH-1/4W
- added R2, R4, R8: 100, MG-Eagle_v1:RES_RESISTOR-PTH-1/4W
- added R3, R7: 10k, MG-Eagle_v1:RES_RESISTOR-PTH-1/4W
- added R5: 220, MG-Eagle_v1:RES_RESISTOR-PTH-1/4W
- added R6: 4k, 1%, MG-Eagle_v1:RES_RESISTOR-PTH-1/4W
- added VRG-2: LM317, MG-Eagle_v1:VRG_LM317_TO-220_VERTICAL
- C1: value (none) -> 100uF, 50V
- LED1: value (none) -> 3mm Green
Connections:
- new net !AMP-SHDN: ASM-1.D10, ASM-3.!SHTDWN, J4.7, J9.5, R1.P2
- new net 24V: C1.+, J1.1, J20.P1, R5.P2, VRG-2.VOUT
- new net 3V: ASM-1.3V, J3.2
- new net 48V: J12.3, J12.4, J13.P2, J14.P2, K1.MAIN-1, K1.MAIN-2, K2.MAIN-1, K2.MAIN-2, VRG-1.VIN@10, VRG-1.VIN@9, VRG-2.VIN
- new net 5V: ASM-1.USB/VBUS, ASM-2.VIN, ASM-3.VCC, ASM-4.VCC, D1.C, J10.1, J10.2, J10.3, J10.4, J15.P1, J16.P1, J19.5, J4.3, J5.9, J8.1, J9.7, JP1.2, K1.COIL-1, K2.COIL-1, LED1.A, U1.VCC, VRG-1.VOUT@1, VRG-1.VOUT@2, VRG-1.VOUT@3, VRG-1.VOUT@4
- new net ADJ: R5.P1, R6.P2, VRG-2.ADJ
- new net CRNT-MON: ASM-1.A0, ASM-4.OUT, J19.1, J3.5
- new net DFU: ASM-1.DFU, J3.16
- new net ENCODER-A: ASM-1.RX0, J3.14
- new net ENCODER-B: ASM-1.TX1, J3.15
- new net ENCODER-SW: ASM-1.D11, J4.6
- new net FAN-CTRL: ASM-1.D6, J4.9, R8.P1
- new net GND: ASM-1.GND@4, ASM-2.GND@14, ASM-2.GND@27, ASM-3.GND, ASM-4.GND, C1.-, J11.1, J11.2, J11.3, J11.4, J18.1, J19.4, J3.4, J5.10, J7.14, J8.2, J9.6, JP2.2, JP3.2, JP4.2, JP5.2, JP6.2, JP7.1, JP8.1, Q1.S, Q2.S, R1.P1, R3.P2, R6.P1, R7.P2, U1.GND, VRG-1.GND@5, VRG-1.GND@6, VRG-1.GND@7, VRG-1.GND@8
- new net I2C-SCL: ASM-1.SCL, J4.11, J5.12, U1.SCL
- new net I2C-SDA: ASM-1.SDA, J4.12, J5.13, U1.SDA
- new net K1-NC: J13.P1, K1.NC-1, K1.NC-2
- new net K2-NC: J14.P1, K2.NC-1, K2.NC-2
- new net LED-DATA: ASM-1.D12, J4.5
- new net MIST-CTRL: ASM-1.D5, J4.10, R2.P1
- new net MIST-VIN: ASM-4.VIN-, J13.P3, J14.P3, J17.1, J19.3, K1.NO-1, K1.NO-2
- new net N$1: ASM-1.!RESET, J3.1
- new net N$10: D1.A, J15.P2, J16.P2, K1.COIL-2, K2.COIL-2, Q1.D, R4.P1
- new net N$11: Q1.G, R2.P2, R3.P1
- new net N$12: J1.2, J20.P2, Q2.D
- new net N$13: LED1.C, R4.P2
- new net N$14: ASM-3.L-IN, J9.3, JP7.2
- new net N$15: ASM-3.R-IN, J9.2, JP8.2
- new net N$16: ASM-4.VIN+, J19.2, K2.NO-1, K2.NO-2
- new net N$17: Q2.G, R7.P1, R8.P2
- new net N$2: ASM-1.AREF, J3.3
- new net N$20: ASM-1.D9, J4.8
- new net N$24: ASM-1.D13, J4.4
- new net N$25: ASM-1.EN, J4.2
- new net N$26: ASM-2.ACT, J7.13
- new net N$27: J12.1, VRG-1.R.C.
- new net N$28: ASM-2.R-GND, J8.11, JP5.1
- new net N$29: J12.2, VRG-1.TRIM
- new net N$3: J5.1, U1.GPB0
- new net N$30: ASM-2.TX, J8.5
- new net N$31: ASM-2.RX, J8.6
- new net N$32: J6.9, U1.INTA
- new net N$33: J6.10, U1.INTB
- new net N$34: J6.11, JP1.1, U1.!RESET
- new net N$35: J6.12, JP2.1, U1.A2
- new net N$36: J6.13, JP3.1, U1.A1
- new net N$37: J6.14, JP4.1, U1.A0
- new net N$38: ASM-2.UART/GPIO_SEL, J8.7
- new net N$4: J5.2, U1.GPB1
- new net N$44: ASM-2.L-GND, J8.14, JP6.1
- new net N$5: ASM-1.A1, J3.6
- new net N$6: ASM-1.A2, J3.7
- new net N$7: ASM-1.A3, J3.8
- new net N$8: ASM-1.A4, J3.9
- new net N$9: ASM-1.A5, J3.10
- new net SFX-0: ASM-2.0, J6.7, J7.2, U1.GPA1
- new net SFX-1: ASM-2.1, J6.6, J7.3, U1.GPA2
- new net SFX-10: ASM-2.10, J5.5, J7.12, U1.GPB4
- new net SFX-2: ASM-2.2, J6.5, J7.4, U1.GPA3
- new net SFX-3: ASM-2.3, J6.4, J7.5, U1.GPA4
- new net SFX-4: ASM-2.4, J6.3, J7.6, U1.GPA5
- new net SFX-5: ASM-2.5, J6.2, J7.7, U1.GPA6
- new net SFX-6: ASM-2.6, J6.1, J7.8, U1.GPA7
- new net SFX-7: ASM-2.7, J5.8, J7.9, U1.GPB7
- new net SFX-8: ASM-2.8, J5.7, J7.10, U1.GPB6
- new net SFX-9: ASM-2.9, J5.6, J7.11, U1.GPB5
- new net SFX-LOUT: ASM-2.L+OUT, ASM-3.L+IN, J8.13, J9.4
- new net SFX-ROUT: ASM-2.R+OUT, ASM-3.R+IN, J8.12, J9.1
- new net SFX-RST: ASM-2.!RESET, J6.8, J7.1, U1.GPA0
- new net SFX-VOL-N: ASM-2.VOL-, J5.3, J8.9, U1.GPB2
- new net SFX-VOL-P: ASM-2.VOL+, J5.4, J8.8, U1.GPB3
- new net SPI-MISO: ASM-1.MISO, J3.13
- new net SPI-MOSI: ASM-1.MOSI, J3.12
- new net SPI-SCK: ASM-1.SCK, J3.11
- new net USB/VBUS: ASM-2.USB/VBUS, J8.3
- new net VBAT: ASM-1.VBAT, J4.1
Other:
- note added: "24V Fan"
- note added: "48V to 5V DC Converter"
- note added: "Dual Relays to distribute the large DC current draw"
- note added: "If there's noise due to grounding audio to the GND plane, cut the jumpers and run GND fly-wires to audio amp"
- note added: "If there's noise on the GND plane cut the jumpers and run GND fly-wires to audio amp"
- note added: "Jumpers allow these lines to be easily cut and re-rounded with flywires from the breakout pads"
- note added: "LM317 requires heatsink"
- note added: "Mister Control"
- note added: "Mister draws 4.4A @ 48V (212W)"
- note added: "Optional: Strong Pull-down Res to keep the amp in Shut Down mode during power on to avoid pops"
- note added: "Rotary Encoder Connector"
- note added: "Speakers wired to screw terminals on Amp board"
- note added: "Vout = 1.25 * (1 + (R5/R6) )"
