File: hardware/elec/eagle-9.5.1/HUM-ASM-001/HUM-ASM-001.sch (EAGLE design)
At the start: 73 parts, among them J1 B2B-XH-AM(LF)(SN), J2 75869-131LF, J22 75869-131LF, J23 75869-131LF, K1 7-1393239-7, K2 7-1393239-7, Q1 IRLB8721PBF, Q2 IRLB8721PBF, U1 MCP23017-E/SP

Commit message: * Removed unneeded components (Breakout connectors and Jumpers) * Laid 5V and GND planes
Parts:
- removed C3: 100uF, 50V, MG-Eagle_v1:CAP_THT_POL-E-035X080MM
- removed J24, J25: (no value), MG-Eagle_v1:CON_HEADER_1X6NO_SILK_FEMALE_PTH
- removed J5, J6: (no value), MG-Eagle_v1:CON_HEADER_1X14
- removed JP1, JP2, JP3, JP4, JP5, JP6: CON_JUMPER_PAD-2-NC_BY_TRACE, MG-Eagle_v1:CON_JUMPER_PAD-2-NC_BY_TRACE
- removed THM-1: 532702B02500G, MG-Eagle_v1:THM_HEATSINK_2-PIN
Connections:
- removed net N$28: ASM-2.R-GND, J8.11, JP5.1
- removed net N$32: J6.9, U1.INTA
- removed net N$33: J6.10, U1.INTB
- removed net N$34: J6.11, JP1.1, U1.!RESET
- removed net N$35: J6.12, JP2.1, U1.A2
- removed net N$36: J6.13, JP3.1, U1.A1
- removed net N$37: J6.14, JP4.1, U1.A0
- removed net N$44: ASM-2.L-GND, J8.14, JP6.1
- net 5V: now also U1.!RESET; no longer C3.+, J24.1, J24.2, J25.1, J25.2, J5.9, JP1.2
- net GND: now also ASM-2.L-GND, ASM-2.R-GND, J8.11, J8.14, U1.A0, U1.A1, U1.A2; no longer C3.-, J24.5, J24.6, J25.5, J25.6, J5.10, JP2.2, JP3.2, JP4.2, JP5.2, JP6.2
- net I2C-SCL: no longer J5.12
- net I2C-SDA: no longer J5.13
- net N$3: no longer J5.1
- net N$4: no longer J5.2
- net N$42: no longer J25.3, J25.4
- net N$9: no longer J24.3, J24.4
- net SFX-0: no longer J6.7
- net SFX-1: no longer J6.6
- net SFX-10: no longer J5.5
- net SFX-2: no longer J6.5
- net SFX-3: no longer J6.4
- net SFX-4: no longer J6.3
- net SFX-5: no longer J6.2
- net SFX-6: no longer J6.1
- net SFX-7: no longer J5.8
- net SFX-8: no longer J5.7
- net SFX-9: no longer J5.6
- net SFX-RST: no longer J6.8
- net SFX-VOL-N: no longer J5.3
- net SFX-VOL-P: no longer J5.4
Other:
- note removed: "If there's noise due to grounding audio to the GND plane, cut the jumpers and run GND fly-wires to audio amp"
- moved on the sheet: C2, R10, R9
